File: hardware/Badge-bsides-cdmx-2025-community/Badge-bsides-cdmx-2025.kicad_pcb (KiCad board)
At the start: 2 copper layers, 49.9 x 109.8 mm, 39 parts, among them J1 SWDIO, J3 ADDON, J4 Conn_01x04_Pin, J5 I2C, J6 Conn_01x04_Pin, SW10 SW_Push, SW11 ON, SW2 RESET, SW7 SW_Push, SW8 SW_Push, SW9 SW_Push, U1 PY32F030F28U6TR

Commit message: fix(Hw):sponsor_and_Community_updated
Parts:
- moved C30 10.2 mm to (51.8, 86.6)
- moved D20 9.05 mm to (53.9, 84.0)
- moved J6 5.85 mm to (44.5, 83.1)
Routing:
- net /RX: track 27.3 -> 22.3 mm
- net +3.3V: track 229.2 -> 230.3 mm
- net Net-(D19-DOUT): track 19.6 -> 18.9 mm
- net /SDA: track 67.7 -> 67.2 mm
- net /SWDIO: track 36.3 -> 36.0 mm, vias 0 -> 2

Commit message: feat(Hw):Update_Route
Routing:
- net GND: vias 8 -> 12
Changed lines of the file:
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@@
 	)
 	(via
-		(at 46.57 51.86)
+		(at 49.99 79.13)
 		(size 0.6)
 		(drill 0.3)
@@
 	)
 	(via
-		(at 48.32 46.41)
+		(at 46.57 51.86)
 		(size 0.6)
 		(drill 0.3)
@@
 	)
 	(via
-		(at 61.79 70.42)
+		(at 49.99 78.13)
 		(size 0.6)
 		(drill 0.3)
@@
 	)
 	(via
-		(at 48.33 47.92)
+		(at 48.32 46.41)
 		(size 0.6)
 		(drill 0.3)
@@
 	)
 	(via
-		(at 62.51 70.42)
+		(at 61.79 70.42)
 		(size 0.6)
 		(drill 0.3)
@@
 	)
 	(via
+		(at 48.33 47.92)
+		(size 0.6)
+		(drill 0.3)
+		(layers "F.Cu" "B.Cu")
+		(free yes)
+		(net 1)
+	)
+	(via
+		(at 62.51 70.42)
+		(size 0.6)
+		(drill 0.3)
+		(layers "F.Cu" "B.Cu")
+		(free yes)
+		(net 1)
+	)
+	(via
+		(at 48.99 79.13)
+		(size 0.6)
+		(drill 0.3)
+		(layers "F.Cu" "B.Cu")
+		(free yes)
+		(net 1)
+	)
+	(via
 		(at 63.23 70.41)
+		(size 0.6)
+		(drill 0.3)
+		(layers "F.Cu" "B.Cu")
+		(free yes)
+		(net 1)
+	)
+	(via
+		(at 48.99 78.13)
 		(size 0.6)
 		(drill 0.3)
@@
 	)
 	(segment
+		(start 59.04 79.595666)
+		(end 58.581333 80.054333)
+		(width 0.2)
+		(layer "B.Cu")
+		(net 11)
+	)
+	(segment
+		(start 58.581333 80.054333)
+		(end 46.804333 80.054333)
+		(width 0.2)
+		(layer "B.Cu")
+		(net 11)
+	)
+	(segment
+		(start 44.161333 64.16)
+		(end 37.328666 64.16)
+		(width 0.2)
+		(layer "B.Cu")
+		(net 11)
+	)
+	(segment
 		(start 45.98 65.978667)
 		(end 44.161333 64.16)
@@
 	)
 	(segment
-		(start 45.98 79.733)
+		(start 45.98 79.23)
 		(end 45.98 65.978667)
 		(width 0.2)
@@
 	)
 	(segment
-		(start 44.161333 64.16)
-		(end 37.328666 64.16)
-		(width 0.2)
-		(layer "B.Cu")
-		(net 11)
-	)
-	(segment
-		(start 58.581333 80.054333)
-		(end 46.301333 80.054333)
-		(width 0.2)
-		(layer "B.Cu")
-		(net 11)
-	)
-	(segment
-		(start 46.301333 80.054333)
-		(end 45.98 79.733)
-		(width 0.2)
-		(layer "B.Cu")
-		(net 11)
-	)
-	(segment
-		(start 59.04 79.595666)
-		(end 58.581333 80.054333)
+		(start 46.804333 80.054333)
+		(end 45.98 79.23)
 		(width 0.2)
 		(layer "B.Cu")
@@
 	)
 	(segment
-		(start 79.806333 74.486333)
-		(end 79.806333 75.244333)
+		(start 66.97 73.99)
+		(end 79.31 73.99)
+		(width 0.2)
+		(layer "F.Cu")
+		(net 18)
+	)
+	(segment
+		(start 79.31 73.99)
+		(end 80.18 74.86)
 		(width 0.2)
 		(layer "F.Cu")
@@
 	)
 	(segment
-		(start 79.31 73.99)
-		(end 79.806333 74.486333)
+		(start 80.18 74.86)
+		(end 80.18 75.46)
 		(width 0.2)
 		(layer "F.Cu")
 		(net 18)
 	)
-	(segment
-		(start 66.97 73.99)
-		(end 79.31 73.99)
-		(width 0.2)
-		(layer "F.Cu")
+	(via
+		(at 63.47 74.06)
+		(size 0.6)
+		(drill 0.3)
+		(layers "F.Cu" "B.Cu")
 		(net 18)
 	)
 	(via
-		(at 63.47 74.06)
+		(at 58.764265 74.065735)
 		(size 0.6)
 		(drill 0.3)
@@
 	)
 	(via
-		(at 58.764265 74.065735)
-		(size 0.6)
-		(drill 0.3)
-		(layers "F.Cu" "B.Cu")
-		(net 18)
-	)
-	(via
 		(at 66.97 73.99)
 		(size 0.6)
 		(drill 0.3)
 		(layers "F.Cu" "B.Cu")
-		(net 18)
-	)
-	(segment
-		(start 79.806333 75.244333)
-		(end 79.806333 77.784333)
-		(width 0.2)
-		(layer "B.Cu")
 		(net 18)
 	)
@@
 	)
 	(segment
+		(start 80.17 75.47)
+		(end 80.17 77.784333)
+		(width 0.2)
+		(layer "B.Cu")
+		(net 18)
+	)
+	(segment
 		(start 59.04 74.34147)
 		(end 58.764265 74.065735)
@@
 		(width 0.2)
 		(layer "B.Cu")
+		(net 18)
+	)
+	(segment
+		(start 80.18 75.46)
+		(end 80.17 75.47)
+		(width 0.2)
+		(layer "B.Cu")

Commit message: fix(Hw):Labels_Updated
Parts:
- D19, D20: value WS2812B -> SK6812MINI-E
- R3: value 1K -> 470R
Connections:
- U1 pad 21: (no net) -> GND
Changed lines of the file:
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@@
 			(layers "*.Cu")
 			(remove_unused_layers no)
+			(net 1 "GND")
+			(pinfunction "VSS")
+			(pintype "bidirectional")
 		)
 		(pad "21" thru_hole circle
@@
 			(layers "*.Cu")
 			(remove_unused_layers no)
+			(net 1 "GND")
+			(pinfunction "VSS")
+			(pintype "bidirectional")
 		)
 		(pad "21" smd rect
@@
 			(property pad_prop_heatsink)
 			(layers "F.Cu")
+			(net 1 "GND")
+			(pinfunction "VSS")
+			(pintype "bidirectional")
 			(zone_connect 2)
 		)
@@
 			(property pad_prop_heatsink)
 			(layers "B.Cu" "B.Mask")
+			(net 1 "GND")
+			(pinfunction "VSS")
+			(pintype "bidirectional")
 			(zone_connect 2)
 		)
@@
 			(layers "*.Cu")
 			(remove_unused_layers no)
+			(net 1 "GND")
+			(pinfunction "VSS")
+			(pintype "bidirectional")
 		)
 		(pad "21" thru_hole circle
@@
 			(layers "*.Cu")
 			(remove_unused_layers no)
+			(net 1 "GND")
+			(pinfunction "VSS")
+			(pintype "bidirectional")
 		)
 		(embedded_fonts no)
@@
 			)
 		)
-		(property "Value" "WS2812B"
+		(property "Value" "SK6812MINI-E"
 			(at 7.26 -3.17151 0)
 			(layer "B.Fab")
@@
 			)
 		)
-		(property "LCSC#" "C527089"
+		(property "LCSC#" "C5149201"
 			(at 0 0 0)
 			(unlocked yes)
@@
 			)
 		)
-		(property "manf#" "WS2812B-Mini"
+		(property "manf#" ""
 			(at 0 0 0)
 			(unlocked yes)
@@
 			)
 		)
-		(property "Value" "WS2812B"
+		(property "Value" "SK6812MINI-E"
 			(at 7.26 -3.17151 0)
 			(layer "B.Fab")
@@
 			)
 		)
-		(property "LCSC#" "C527089"
+		(property "LCSC#" "C5149201"
 			(at 0 0 0)
 			(unlocked yes)
@@
 			)
 		)
-		(property "manf#" "WS2812B-Mini"
+		(property "manf#" ""
 			(at 0 0 0)
 			(unlocked yes)
@@
 			)
 		)
-		(property "LCSC#" "C478888"
+		(property "LCSC#" "C66501"
 			(at 0 0 180)
 			(unlocked yes)
@@
 			)
 		)
-		(property "LCSC#" "C14663"
+		(property "LCSC#" "C66501"
 			(at 0 0 90)
 			(unlocked yes)
@@
 			)
 		)
-		(property "Value" "1K"
+		(property "Value" "470R"
 			(at 0 -1.43 0)
 			(layer "B.Fab")
@@
 			)
 		)
-		(property "LCSC#" "C22548"
+		(property "LCSC#" "C114669"
 			(at 0 0 0)
 			(unlocked yes)
@@
 			)
 		)
-		(property "LCSC#" "C14663"
+		(property "LCSC#" "C66501"
 			(at 0 0 90)
 			(unlocked yes)
@@
 			)
 		)
-		(property "LCSC#" "C478888"
+		(property "LCSC#" "C66501"
 			(at 0 0 180)
 			(unlocked yes)
