File: hardware/Badge-bsides-cdmx-2025-community/Badge-bsides-cdmx-2025.kicad_sch (KiCad schematic)
At the start: 31 parts, among them J1 SWDIO, J3 ADDON, J4 Conn_01x04_Pin, J5 I2C, J6 Conn_01x04_Pin, SW10 SW_Push, SW11 ON, SW2 RESET, SW7 SW_Push, SW8 SW_Push, SW9 SW_Push, U1 PY32F030F28U6TR

Commit message: fix(Hw):Labels_Updated
Parts:
- R3: value 1K -> 470R; LCSC# C22548 -> C114669
Connections:
- net GND: now also U1.21 (VSS)
Changed lines of the file:
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@@
 			)
 		)
-		(property "Value" "1K"
+		(property "Value" "470R"
 			(at 34.29 108.585 90)
 			(effects
@@
 			)
 		)
-		(property "LCSC#" "C22548"
+		(property "LCSC#" "C114669"
 			(at 34.29 110.49 0)
 			(effects
@@
 		(pin "12"
 		)
+		(pin "21"
+		)
 		(instances
