File: hardware/Badge-bsides-cdmx-2025-guest/Badge-bsides-cdmx-2025.kicad_sch (KiCad schematic)
At the start: 43 parts, among them J1 SWDIO, J3 ADDON, J4 Conn_01x04_Pin, J5 I2C, J6 Conn_01x04_Pin, P6 USB_C_Plug_USB2.0, Q3 DMG3415U-7, SW10 SW_Push, SW11 ON, SW2 RESET, SW7 SW_Push, SW8 SW_Push, SW9 SW_Push, U1 PY32F030F28U6TR, U6 AP2112K-3.3

Commit message: Auto stash before merge of "main" and "origin/main"
Parts:
- removed C10, C27: 10uF, Capacitor_SMD:C_0603_1608Metric, symbol Device:C_Small
- removed D4: MBR120, Diode_SMD:D_SOD-123F, symbol Diode:MBR340
- removed F3: 750mA, Fuse:Fuse_0603_1608Metric, symbol Device:Fuse_Small
- removed P6: USB_C_Plug_USB2.0, Footprints:C393939, symbol HunterCat-NFC-rescue:USB_C_Plug_USB2.0-Connector
- removed Q3: DMG3415U-7, Package_TO_SOT_SMD:SOT-23, symbol Device:Q_PMOS_GSD
- removed R10: 100K, Resistor_SMD:R_0603_1608Metric, symbol Device:R_Small
- removed R41, R45: 5k1, Resistor_SMD:R_0603_1608Metric, symbol Device:R_Small
- removed U6: AP2112K-3.3, Package_TO_SOT_SMD:SOT-23-5, symbol HunterCat-NFC-rescue:AP2112K-3.3-Regulator_Linear
- SW11: LCSC# - -> C221660; Manufacturer_Part_Number JS102011SAQN -> (none); manf# JS102011SAQN -> (none)
Connections:
- net +3V3 is gone; now on net +3.3V: C26.1, J3.1 (Pin_1), R4.2, R5.2, R6.2, R7.2, R8.2
- net +3.3V: now also C33.1, SW11.3 (A)
- net +BATT: now also BT3.1 (+), SW11.2 (B); no longer BT3.2 (+)
- net GND: now also BT4.2 (-); no longer BT4.1 (-)
- net GPIO1: now also U1.11 (PB7); no longer U1.3 (PA7)
- net GPIO2: now also U1.12 (PF4/BOOT0); no longer U1.5 (PA12)
- net NEO: now also U1.3 (PA7)
- net RX: now also J6.3 (Pin_3), J6.4 (Pin_4); no longer J4.3 (Pin_3), J4.4 (Pin_4)
- net TX: now also J4.3 (Pin_3), J4.4 (Pin_4); no longer J6.3 (Pin_3), J6.4 (Pin_4)
- net VBUS: no longer C33.1
- net LED1: no longer names the net of U1.10 (PB6)
- new net: BT3.2 (-), BT4.1 (+)
Other:
- moved on the sheet: C26, C33, C6, C67, C68, C69, C70, R4, R5, R6, R7, R8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

Commit message: fix(Hw):Labels_Updated
Parts:
- R12: value 1K -> 470R; LCSC# C22548 -> C114669
Connections:
- net GND: now also U1.21 (VSS)
Changed lines of the file:
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@@
 		)
 	)
-	(label "NEO"
-		(at 212.09 49.53 180)
-		(effects
-			(font
-				(size 1.27 1.27)
-			)
-			(justify right bottom)
-		)
-	)
 	(label "GPIO1"
 		(at 128.27 105.41 180)
@@
 		(pin "12"
 		)
+		(pin "21"
+		)
 		(instances
 			(project ""
@@
 			)
 		)
-		(property "Value" "1K"
+		(property "Value" "470R"
 			(at 26.67 111.125 90)
 			(effects
@@
 			)
 		)
-		(property "LCSC#" "C22548"
+		(property "LCSC#" "C114669"
 			(at 26.67 113.03 0)
 			(effects
