File: hardware/Badge-bsides-cdmx-2025-sponsor/Badge-bsides-cdmx-2025.kicad_pcb (KiCad board)
At the start: 2 copper layers, 49.9 x 109.8 mm, 53 parts, among them J1 SWDIO, J3 ADDON, J4 Conn_01x04_Pin, J5 I2C, J6 Conn_01x04_Pin, P6 USB_C_Plug_USB2.0, Q3 DMG3415U-7, SW10 SW_Push, SW11 ON, SW2 RESET, SW7 SW_Push, SW8 SW_Push, SW9 SW_Push, U1 PY32F030F28U6TR, U6 AP2112K-3.3

Commit message: Auto stash before merge of "main" and "origin/main"
Parts:
- removed C10: 10uF, Capacitor_SMD:C_0603_1608Metric
- removed C33: 100nF, Capacitor_SMD:C_0603_1608Metric
- removed D4: MBR120, Diode_SMD:D_SOD-123F
- removed F3: 750mA, Fuse:Fuse_0603_1608Metric
- removed P6: USB_C_Plug_USB2.0, Footprints:C393939
- removed Q3: DMG3415U-7, Package_TO_SOT_SMD:SOT-23
- removed R10: 100K, Resistor_SMD:R_0603_1608Metric
- removed R41, R45: 5k1, Resistor_SMD:R_0603_1608Metric
- removed U6: AP2112K-3.3, Package_TO_SOT_SMD:SOT-23-5
- removed kibuzzard-6841D7B6: G***, kibuzzard-6841D7B6
- removed kibuzzard-6841DB7D: G***, kibuzzard-6841DB7D
- removed kibuzzard-6841DDA6: G***, kibuzzard-6841DDA6
- removed kibuzzard-6841DDB3: G***, kibuzzard-6841DDB3
- added kibuzzard-684316B7: G***, kibuzzard-684316B7, B.Cu at (130.5, 90.1)
- added kibuzzard-684316C2: G***, kibuzzard-684316C2, B.Cu at (160.6, 90.0)
- added kibuzzard-684316CB: G***, kibuzzard-684316CB, B.Cu at (119.4, 100.2)
- added kibuzzard-684316D5: G***, kibuzzard-684316D5, B.Cu at (119.2, 111.2)
- D19, D20: value WS2812B -> SK6812MINI-E
- moved C27 28.7 mm to (126.5, 102.4), turned to 90 degrees
- moved C26 6.38 mm to (128.0, 102.4), turned to 90 degrees
- moved J4 0.14 mm to (163.2, 93.8)
- moved J6 0.14 mm to (127.6, 93.7)
Connections:
- C27 pad 1: VBUS -> +3.3V
- SW11 pad 2: Net-(D4-K) -> +BATT
- SW11 pad 3: Net-(SW11-A) -> +3.3V
Routing:
- net VBUS: track 74.7 -> 0.00 mm, vias 3 -> 0
- net Net-(SW11-A): track 14.8 -> 0.00 mm
- net Net-(F3-Pad1): track 10.8 -> 0.00 mm
- net +3.3V: track 185.9 -> 195.9 mm
- net +BATT: track 14.6 -> 24.5 mm
- net Net-(D4-K): track 9.51 -> 0.00 mm
- net Net-(P6-CC): track 7.73 -> 0.00 mm
- net Net-(P6-VCONN): track 6.86 -> 0.00 mm
- net GND: vias 16 -> 18

Commit message: fix(Hw):sponsor_and_Community_updated
Parts:
- moved J4 0.79 mm to (163.2, 93.0)
- moved J6 0.76 mm to (127.6, 93.0)
Changed lines of the file:
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@@
 		(tenting front back)
 		(pcbplotparams
-			(layerselection 0x00000000_00000000_55555555_555555f0)
+			(layerselection 0x00000000_00000000_55555555_575555d0)
 			(plot_on_all_layers_selection 0x00000000_00000000_00000000_00000000)
 			(disableapertmacros no)
@@
 	(footprint "Connector_PinSocket_2.54mm:PinSocket_1x04_P2.54mm_Horizontal"
 		(layer "B.Cu")
-		(at 127.61 93.74)
+		(at 127.61 92.983133)
 		(descr "Through hole angled socket strip, 1x04, 2.54mm pitch, 8.51mm socket length, single row (from Kicad 4.0.7), script generated")
 		(tags "Through hole angled socket strip THT 1x04 2.54mm single row")
@@
 	(footprint "Connector_PinHeader_2.54mm:PinHeader_1x04_P2.54mm_Horizontal"
 		(layer "B.Cu")
-		(at 163.17 93.774)
+		(at 163.17 92.983133)
 		(descr "Through hole angled pin header, 1x04, 2.54mm pitch, 6mm pin length, single row")
 		(tags "Through hole angled pin header THT 1x04 2.54mm single row")
@@
 	(gr_curve
 		(pts
+			(xy 162.31 37.13) (xy 161.298755 37.13) (xy 160.387083 37.739159) (xy 160.000096 38.673429)
+		)
+		(stroke
+			(width 0.2)
+			(type default)
+		)
+		(layer "B.SilkS")
+	)
+	(gr_line
+		(start 167.310162 40.686493)
+		(end 167.310162 142.596883)
+		(stroke
+			(width 0.2)
+			(type default)
+		)
+		(layer "B.SilkS")
+	)
+	(gr_curve
+		(pts
+			(xy 160.000096 38.673429) (xy 159.613109 39.607698) (xy 159.827018 40.683088) (xy 160.542076 41.398146)
+		)
+		(stroke
+			(width 0.2)
+			(type default)
+		)
+		(layer "B.SilkS")
+	)
+	(gr_curve
+		(pts
+			(xy 164.810223 39.630222) (xy 164.810223 38.967122) (xy 164.546807 38.331181) (xy 164.077925 37.862298)
+		)
+		(stroke
+			(width 0.2)
+			(type default)
+		)
+		(layer "B.SilkS")
+	)
+	(gr_curve
+		(pts
+			(xy 119.418622 144.604103) (xy 118.326972 144.604103) (xy 117.411402 143.723743) (xy 117.411402 142.596883)
+		)
+		(stroke
+			(width 0.2)
+			(type default)
+		)
+		(layer "B.SilkS")
+	)
+	(gr_curve
+		(pts
+			(xy 167.310162 142.596883) (xy 167.345362 143.723743) (xy 166.465022 144.604103) (xy 165.338162 144.604103)
+		)
+		(stroke
+			(width 0.2)
+			(type default)
+		)
+		(layer "B.SilkS")
+	)
+	(gr_curve
+		(pts
+			(xy 161.429362 34.805693) (xy 164.669082 34.805693) (xy 167.310162 37.446773) (xy 167.310162 40.686493)
+		)
+		(stroke
+			(width 0.2)
+			(type default)
+		)
+		(layer "B.SilkS")
+	)
+	(gr_curve
+		(pts
+			(xy 160.542076 41.398146) (xy 161.257135 42.113205) (xy 162.332525 42.327113) (xy 163.266794 41.940126)
+		)
+		(stroke
+			(width 0.2)
+			(type default)
+		)
+		(layer "B.SilkS")
+	)
+	(gr_line
+		(start 123.292202 34.805693)
+		(end 161.429362 34.805693)
+		(stroke
+			(width 0.2)
+			(type default)
+		)
+		(layer "B.SilkS")
+	)
+	(gr_line
+		(start 117.411402 142.596883)
+		(end 117.411402 40.686493)
+		(stroke
+			(width 0.2)
+			(type default)
+		)
+		(layer "B.SilkS")
+	)
+	(gr_curve
+		(pts
+			(xy 163.266794 41.940126) (xy 164.201063 41.55314) (xy 164.810223 40.641468) (xy 164.810223 39.630222)
+		)
+		(stroke
+			(width 0.2)
+			(type default)
+		)
+		(layer "B.SilkS")
+	)
+	(gr_line
+		(start 165.338162 144.604103)
+		(end 119.418622 144.604103)
+		(stroke
+			(width 0.2)
+			(type default)
+		)
+		(layer "B.SilkS")
+	)
+	(gr_curve
+		(pts
+			(xy 164.077925 37.862298) (xy 163.609042 37.393415) (xy 162.973101 37.13) (xy 162.31 37.13)
+		)
+		(stroke
+			(width 0.2)
+			(type default)
+		)
+		(layer "B.SilkS")
+	)
+	(gr_curve
+		(pts
+			(xy 117.411402 40.686493) (xy 117.411402 37.446773) (xy 120.052482 34.805693) (xy 123.292202 34.805693)
+		)
+		(stroke
+			(width 0.2)
+			(type default)
+		)
+		(layer "B.SilkS")
+	)
+	(gr_curve
+		(pts
 			(xy 164.067763 37.865415) (xy 163.59888 37.396532) (xy 162.962939 37.133117) (xy 162.299838 37.133117)
 		)
@@
 	)
 	(segment
-		(start 127.61 86.12)
-		(end 127.61 88.66)
-		(width 0.2)
-		(layer "B.Cu")
-		(net 13)
-	)
-	(segment
-		(start 130.65 85.32)
-		(end 129.74 85.32)
+		(start 127.61 85.363133)
+		(end 127.61 87.903133)
 		(width 0.2)
 		(layer "B.Cu")
@@
 	)
 	(segment
-		(start 130.68 85.35)
-		(end 130.65 85.32)
+		(start 130.956867 85.363133)
+		(end 130.97 85.35)
 		(width 0.2)
 		(layer "B.Cu")
@@
 	(segment
 		(start 140.6 85.35)
-		(end 130.68 85.35)
+		(end 130.97 85.35)
 		(width 0.2)
 		(layer "B.Cu")
@@
 	)
 	(segment
-		(start 128.94 86.12)
-		(end 129.74 85.32)
-		(width 0.2)
-		(layer "B.Cu")
-		(net 13)
-	)
-	(segment
-		(start 127.61 86.12)
-		(end 128.94 86.12)
+		(start 144.5 88.9)
+		(end 144.85 88.55)
 		(width 0.2)
 		(layer "B.Cu")
@@
 	)
 	(segment
-		(start 144.5 88.9)
-		(end 144.85 88.55)
+		(start 127.61 85.363133)
+		(end 130.956867 85.363133)
 		(width 0.2)
 		(layer "B.Cu")
@@
 	)
 	(segment
-		(start 163.17 86.154)
-		(end 163.17 88.694)
-		(width 0.2)
-		(layer "B.Cu")
-		(net 19)
-	)
-	(segment
-		(start 163.17 86.154)
-		(end 161.87 86.154)
+		(start 163.17 85.363133)
+		(end 145.236867 85.363133)
 		(width 0.2)
 		(layer "B.Cu")
@@
 	)
 	(segment
-		(start 161.87 86.154)
-		(end 161.73 86.014)
+		(start 144.586 86.014)
+		(end 144.1 86.5)
 		(width 0.2)
 		(layer "B.Cu")
@@
 	)
 	(segment
-		(start 144.586 86.014)
-		(end 144.1 86.5)
+		(start 145.236867 85.363133)
+		(end 144.586 86.014)
 		(width 0.2)
 		(layer "B.Cu")
@@
 	)
 	(segment
-		(start 161.73 86.014)
-		(end 144.586 86.014)
+		(start 163.17 87.903133)
+		(end 163.17 85.363133)
 		(width 0.2)
 		(layer "B.Cu")

Commit message: fix(Hw):Ground_and_neopixel_resistor(sponsor)
Parts:
- R3: value 1K -> 470
Connections:
- U1 pad 21: (no net) -> GND
Changed lines of the file:
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@@
 			(layers "*.Cu")
 			(remove_unused_layers no)
+			(net 1 "GND")
+			(pinfunction "VSS")
+			(pintype "bidirectional")
 		)
 		(pad "21" thru_hole circle
@@
 			(layers "*.Cu")
 			(remove_unused_layers no)
+			(net 1 "GND")
+			(pinfunction "VSS")
+			(pintype "bidirectional")
 		)
 		(pad "21" smd rect
@@
 			(property pad_prop_heatsink)
 			(layers "F.Cu")
+			(net 1 "GND")
+			(pinfunction "VSS")
+			(pintype "bidirectional")
 			(zone_connect 2)
 		)
@@
 			(property pad_prop_heatsink)
 			(layers "B.Cu" "B.Mask")
+			(net 1 "GND")
+			(pinfunction "VSS")
+			(pintype "bidirectional")
 			(zone_connect 2)
 		)
@@
 			(layers "*.Cu")
 			(remove_unused_layers no)
+			(net 1 "GND")
+			(pinfunction "VSS")
+			(pintype "bidirectional")
 		)
 		(pad "21" thru_hole circle
@@
 			(layers "*.Cu")
 			(remove_unused_layers no)
+			(net 1 "GND")
+			(pinfunction "VSS")
+			(pintype "bidirectional")
 		)
 		(embedded_fonts no)
@@
 			)
 		)
-		(property "Value" "1K"
+		(property "Value" "470"
 			(at 0 -1.43 90)
 			(layer "B.Fab")
@@
 			)
 		)
-		(property "LCSC#" "C22548"
+		(property "LCSC#" "C114669"
 			(at 0 0 90)
 			(unlocked yes)
@@
 			"AAAAAAAAAAAAAAAAAAAAAAAAAAAAAAAAAAAAAAAAAAAAAAAAAAAAAAAAAAAAAAAAAAAAAAAAAAAA"
 			"AAAAAAAAAAAAAAAAAAAAAAAAAAAAAAAAAAAAAAAAAAAAAAAAAAAAAAAAAAAAAAAAAAAAAAAAAAAA"
-			"AAAAAAAAAAAAAAAAAAAAAAAAAAAAAAAAAAAAAA=="
+			"AAAAAAAAAAAAAAAAAAAAAAAAAAAAAAAAAAAAAAcAAAAAAAAAAAAAAAAAAAAAAAAAAAAAAAQAAAAA"
+			"AAAAAACssV4CAAAAAAAAAAAAAAAAAAAAAAAABwAAAAAAAAAAAAAAAAAAAAAAAAAAAAAABAAAAAAA"
+			"AAAAAI6xXgIAAAAAAAAAAAAAAAAAAAAAAAAHAAAAAAAAAAAAAAAAAAAAAAAAAAAAAAAEAAAAAAAA"
+			"AAAAAAAAAAAAAAAAAAAAAAAAAAAAAAAAAAcAAAAAAAAAAAAAAAAAAAAAAAAAAAAAAAQAAAAAAAAA"
+			"AACOsV4CAAAAAAAAAAAAAAAAAAAAAAAABwAAAAAAAAAAAAAAAAAAAAAAAAAAAAAABAAAAAAAAAAA"
+			"AKyxXgIAAAAAAAAAAAAAAAAAAAAAAAAHAAAAAAAAAAAAAAAAAAAAAAAAAAAAAAABAAAAAAAAAAAA"
+			"rLFeAgAAAAAAAAAAAAAAAAAAAAAAAAcAAAAAAAAAAAAAAAAAAAAAAAAAAAAAAAEAAAAAAAAAAACO"
+			"sV4CAAAAAAAAAAAAAAAAAAAAAAAABwAAAAAAAAAAAAAAAAAAAAAAAAAAAAAAAQAAAAAAAAAAAAAA"
+			"AAAAAAAAAAAAAAAAAAAAAAAAAAAAAAAAAAAAAAAAAAAAAAAAAAAAAAAAAAAAAAAAAAAAAAAAAAAA"
+			"AAAAAAAAAAAAAAAAAAAAAAAAAAAAAAAAAAAAXJnSdwCZAIAAAKqxXgIAAAAAAAAAAAAAAAAAAAAA"
+			"AAAHAAAAAAAAAAAAAAAAAAAAAAAAAAAAAAAIAAAAAAAAAAAAurFeAgAAAAAAAAAAAAAAAAAAAAAA"
+			"AAcAAAAAAAAAAAAAAAAAAAAAAAAAAAAAAAQAAAAAAAAAAABlAGEAdABoAGUAcgAAAAAAAAAAAAAA"
+			"BwAAAAAAAAAAAAAAAAAAAAAAAAAAAAAABAAAAAAAAAAAALqxXgIAAAAAAAAAAAAAAAAAAAAAAAAH"
+			"AAAAAAAAAAAAAAAAAAAAAAAAAAAAAAAEAAAAAAAAAAAAbwBkAHUAbABlAAAAAAAAAAAAAAAAAAcA"
+			"AAAAAAAAAAAAAAAAAAAAAAAAAAAAAAQAAAAAAAAAAABTAEIAAAAAAAAAAAAAAAAAAAAAAAAABwAA"
+			"AAAAAAAAAAAAAAAAAAAAAAAAAAAABAAAAAAAAAAAADAAAAAAAAAAAAAAAAAAAAAAAAAAAAAHAAAA"
+			"AAAAAAAAAAAAAAAAAAAAAAAAAAAEAAAAAAAAAAAAQQBNAEQAMgAxAAAAAAAAAAAAAAAAAAcAAAAA"
+			"AAAAAAAAAAAAAAAAAAAAAAAAAAQAAAAAAAAAAABhAGQAaQBvAAAAAAAAAAAAAAAAAAAABwAAAAAA"
+			"AAAAAAAAAAAAAAAAAAAAAAAABAAAAAAAAAAAAA=="
 		)
 	)
